Commit message: Success running

File: ouster_slam/urdf/os_sensor.urdf (robot description, URDF)
Before this commit: robot os1_sensor, 4 links, 3 joints
Links:
- removed link os1_imu
- removed link os1_lidar
- removed link os1_sensor
- added link os_imu; visual box size=0.06 0.04 0.02
- added link os_lidar; visual cylinder length=0.07 radius=0.05
- added link os_sensor
Joints:
- removed joint os1_link_joint
- added joint os_link_joint: type fixed, parent os_sensor, child os_lidar, origin xyz=0.0 0.0 0.03618 rpy=0 0 3.14159
- joint imu_link_joint: child os1_imu -> os_imu; parent os1_sensor -> os_sensor
- joint sensor_link_joint: child os1_sensor -> os_sensor
