Commit message: Add rviz config and flip lidar Z axis direction

File: drone_simulation/urdf/drone.urdf (robot description, URDF)
Before this commit: robot iris, 4 links, 3 joints
Joints:
- joint os_link_joint: origin xyz=0.0 0.0 0.03618 rpy=0 0 3.14159 -> xyz=0.0 0.0 0.03618 rpy=0 0 0

Commit message: Success robot_localization with ugly hack

File: drone_simulation/urdf/drone.urdf (robot description, URDF)
Before this commit: robot iris, 4 links, 3 joints
Joints:
- joint os_link_joint: origin xyz=0.0 0.0 0.03618 rpy=0 0 0 -> xyz=0.0 0.0 0.03618 rpy=-1.57 0 0
- joint sensor_link_joint: origin xyz=-0.035 0 0.112 rpy=0 1.570796 0 -> xyz=-0.035 0 -0.112 rpy=0 0 0

Commit message: Connected to HDL graph slam

File: drone_simulation/urdf/drone.urdf (robot description, URDF)
Before this commit: robot iris, 4 links, 3 joints
Joints:
- joint os_link_joint: origin xyz=0.0 0.0 0.03618 rpy=-1.57 0 0 -> xyz=0.0 0.0 0.03618 rpy=0 1.57 0
